Commit message: Adjust manipulator chain to match UR world & tool frames.

File: ur_description/urdf/ur10_robot.urdf.xacro (robot description, xacro)
@@ -12,5 +12,5 @@
     <parent link="world" />
     <child link = "base_link" />
-    <origin xyz="0.0 0.0 0.0" rpy="0.0 0.0 0.0" />
+    <origin xyz="0.0 0.0 0.0" rpy="0.0 0.0 ${pi}" />
   </joint>
 </robot>
